File: GameGirl-dev.sch (KiCad schematic (older format))
At the start: 56 parts, among them J1 USB_C_Receptacle_USB2.0, J2 2.54-connector, SW1 TS-1187, SW10 SKRRAAE, SW2 TS-1187, SW3 TS-1187, SW4 TS-1187, SW5 SKRRAAE, SW6 SKRRAAE, SW7 SKRRAAE, SW8 SKRRAAE, SW9 SKRRAAE, U1 SRV05, U2 STM32F411CEUx, U3 AMS1117-3.3, Y1 Crystal_GND24_Small

Commit message: last modifs before fabrication
Parts:
- D1, D2: footprint LED_SMD:LED_0805_2012Metric -> LED_SMD:LED_0603_1608Metric
- J1: LCSC (none) -> C319148
- SW1, SW2, SW3, SW4: LCSC (none) -> C318884
- SW10, SW5, SW6, SW7, SW8, SW9: LCSC (none) -> C97437
- U1: LCSC (none) -> C85364
- Y1: LCSC (none) -> C9006
Changed lines of the file:
@@
 F 2 "caca:TS1187ABAB" H 1350 2900 50  0001 C CNN
 F 3 "http://www.apem.com/int/index.php?controller=attachment&id_attachment=1371" H 1350 2900 50  0001 C CNN
+F 4 "C318884" H 1350 2600 50  0001 C CNN "LCSC"
 	1    1350 2600
 	1    0    0    -1
@@
 F 2 "caca:USB_C_Receptacle_XKB_U262-16XN-4BVC11" H 1850 6400 50  0001 C CNN
 F 3 "https://www.usb.org/sites/default/files/documents/usb_type-c.zip" H 1850 6400 50  0001 C CNN
+F 4 "C319148" H 1700 6400 50  0001 C CNN "LCSC"
 	1    1700 6400
 	1    0    0    -1
@@
 F 2 "caca:TS1187ABAB" H 1200 1650 50  0001 C CNN
 F 3 "http://www.apem.com/int/index.php?controller=attachment&id_attachment=1371" H 1200 1650 50  0001 C CNN
+F 4 "C318884" H 1200 1350 50  0001 C CNN "LCSC"
 	1    1200 1350
 	1    0    0    -1
@@
 F 0 "D1" H 5243 895 50  0000 C CNN
 F 1 "LED" H 5243 986 50  0000 C CNN
-F 2 "LED_SMD:LED_0805_2012Metric" H 5250 1150 50  0001 C CNN
+F 2 "LED_SMD:LED_0603_1608Metric" H 5250 1150 50  0001 C CNN
 F 3 "~" H 5250 1150 50  0001 C CNN
 	1    5250 1150
@@
 F 2 "Crystal:Crystal_SMD_3225-4Pin_3.2x2.5mm" H 3400 1050 50  0001 C CNN
 F 3 "~" H 3400 1050 50  0001 C CNN
+F 4 "C9006" H 3400 1050 50  0001 C CNN "LCSC"
 	1    3400 1050
 	1    0    0    -1
@@
 F 2 "caca:SKRR" H 10150 3100 50  0001 C CNN
 F 3 "http://www.apem.com/int/index.php?controller=attachment&id_attachment=1371" H 10150 3100 50  0001 C CNN
+F 4 "C97437" H 10150 2800 50  0001 C CNN "LCSC"
 	1    10150 2800
 	1    0    0    -1
@@
 F 2 "caca:SKRR" H 10150 4600 50  0001 C CNN
 F 3 "http://www.apem.com/int/index.php?controller=attachment&id_attachment=1371" H 10150 4600 50  0001 C CNN
+F 4 "C97437" H 10150 4300 50  0001 C CNN "LCSC"
 	1    10150 4300
 	1    0    0    -1
@@
 F 2 "caca:SKRR" H 10150 6150 50  0001 C CNN
 F 3 "http://www.apem.com/int/index.php?controller=attachment&id_attachment=1371" H 10150 6150 50  0001 C CNN
+F 4 "C97437" H 10150 5850 50  0001 C CNN "LCSC"
 	1    10150 5850
 	1    0    0    -1
@@
 F 2 "caca:SKRR" H 8400 3000 50  0001 C CNN
 F 3 "http://www.apem.com/int/index.php?controller=attachment&id_attachment=1371" H 8400 3000 50  0001 C CNN
+F 4 "C97437" H 8400 2700 50  0001 C CNN "LCSC"
 	1    8400 2700
 	1    0    0    -1
@@
 F 2 "caca:TS1187ABAB" H 4000 7150 50  0001 C CNN
 F 3 "http://www.apem.com/int/index.php?controller=attachment&id_attachment=1371" H 4000 7150 50  0001 C CNN
+F 4 "C318884" H 4000 6850 50  0001 C CNN "LCSC"
 	1    4000 6850
 	1    0    0    -1
@@
 F 2 "caca:TS1187ABAB" H 5750 7150 50  0001 C CNN
 F 3 "http://www.apem.com/int/index.php?controller=attachment&id_attachment=1371" H 5750 7150 50  0001 C CNN
+F 4 "C318884" H 5750 6850 50  0001 C CNN "LCSC"
 	1    5750 6850
 	1    0    0    -1
@@
 F 2 "caca:SKRR" H 8450 4600 50  0001 C CNN
 F 3 "http://www.apem.com/int/index.php?controller=attachment&id_attachment=1371" H 8450 4600 50  0001 C CNN
+F 4 "C97437" H 8450 4300 50  0001 C CNN "LCSC"
 	1    8450 4300
 	1    0    0    -1
@@
 F 2 "caca:SKRR" H 8450 6150 50  0001 C CNN
 F 3 "http://www.apem.com/int/index.php?controller=attachment&id_attachment=1371" H 8450 6150 50  0001 C CNN
+F 4 "C97437" H 8450 5850 50  0001 C CNN "LCSC"
 	1    8450 5850
 	1    0    0    -1
@@
 F 0 "D2" H 5243 1545 50  0000 C CNN
 F 1 "LED" H 5243 1636 50  0000 C CNN
-F 2 "LED_SMD:LED_0805_2012Metric" H 5250 1800 50  0001 C CNN
+F 2 "LED_SMD:LED_0603_1608Metric" H 5250 1800 50  0001 C CNN
 F 3 "~" H 5250 1800 50  0001 C CNN
 	1    5250 1800
@@
 F 2 "Package_TO_SOT_SMD:SOT-23-6" H 1020 3870 50  0001 C CNN
 F 3 "https://www.diodes.com/assets/Datasheets/D3V3XA4B10LP.pdf" H 1600 4300 50  0001 C CNN
+F 4 "C85364" H 1600 4300 50  0001 C CNN "LCSC"
 	1    1600 4300
 	1    0    0    -1
@@
 Wire Wire Line
 	7200 5300 7250 5300
+Text Label 7250 5300 0    50   ~ 0
+~SCR_NRST
 Wire Bus Line
 	5600 4700 5600 5400
-Text Label 7250 5300 0    50   ~ 0
-~SCR_NRST
 $EndSCHEMATC
