File: LCD_Connector.sch (KiCad schematic (older format))
At the start: 3 parts, among them J3 FH28-40S-0.5SH(07)

Commit message: last modifs before fabrication
Parts:
- J3: LCSC (none) -> C424677
Changed lines of the file:
@@
 F 2 "caca:FH2840S05SH07" H 7550 3500 50  0001 C CNN
 F 3 "~" H 7550 3500 50  0001 C CNN
+F 4 "C424677" H 7550 3500 50  0001 C CNN "LCSC"
 	1    7550 3500
 	1    0    0    -1
